Commit message: refactored for state estimation interface

File: go1_sim/go1_description/xacro/robot.xacro (robot description, xacro)
@@ -17,8 +17,8 @@
     <!-- Debug mode will hung up the robot, use "true" or "false" to switch it. -->
     <xacro:if value="$(arg DEBUG)">
-        <link name="world"/>
+        <link name="odom"/>
         <joint name="base_static_joint" type="fixed">
             <origin rpy="0 0 0" xyz="0 0 0"/>
-            <parent link="world"/>
+            <parent link="odom"/>
             <child link="base"/>
         </joint>
@@ -159,5 +159,5 @@
         <pose>0 0 0 0 0 0</pose>
         <visualize>false</visualize>
-        <update_rate>10</update_rate>
+        <update_rate>30</update_rate>
         <ray>
             <scan>
@@ -194,5 +194,5 @@
             <body_name>base_link</body_name>
             <topic_name>odom</topic_name>
-            <!-- <frame_name>world</frame_name> -->
+            <frame_name>odom</frame_name>
             <update_rate>100</update_rate>
         </plugin>
